Commit message: control and simulation launch done

File: description/inertial_macros.xacro (robot description, xacro)
@@ -1,10 +1,6 @@
 <?xml version="1.0"?>
-<!-- <robot xmlns:xacro="http://www.ros.org/wiki/xacro" name="simple_robot"> -->
 <robot xmlns:xacro="http://www.ros.org/wiki/xacro">
     <!-- This file is not a robot in and of itself, it just contains some useful tags that could be included in any robot -->
     <!-- Specify some colours -->
-    <!-- <material name="orange">
-        <color rgba="1 0.3 0.1 1"/>
-    </material> -->
     <!-- Specify some standard inertial calculations https://en.wikipedia.org/wiki/List_of_moments_of_inertia -->
     <!-- These make use of xacro's mathematical functionality -->

File: description/robot.urdf.xacro (robot description, xacro)
@@ -1,8 +1,6 @@
 <?xml version="1.0"?>
 <robot xmlns:xacro="http://www.ros.org/wiki/xacro" name="robot">
-    <!-- <xacro:include filename="example_include.xacro" /> -->
+    <xacro:include filename="gazebo_control.xacro"/>
     <xacro:include filename="robot_core.xacro" />
     <!-- <xacro:include filename="gazebo.xacro"/> -->
-    <!-- <link name="base_link">
-    </link> -->
 </robot>

File: description/robot_core.xacro (robot description, xacro)
@@ -3,5 +3,4 @@
 <robot xmlns:xacro="http://www.ros.org/wiki/xacro">
     <xacro:include filename="inertial_macros.xacro"/>
-    <!-- <xacro:include filename="example_include.xacro"/> -->
     <xacro:property name="chassis_length" value="0.335"/>
     <xacro:property name="chassis_width" value="0.265"/>
@@ -56,5 +55,5 @@
                 <box size="${chassis_length} ${chassis_width} ${chassis_height}"/>
             </geometry>
-            <material name="orange"/>
+            <material name="red"/>
         </visual>
         <collision>
@@ -68,4 +67,7 @@
         </xacro:inertial_box>
     </link>
+    <gazebo reference="chassis">
+        <material>Gazebo/White</material>
+    </gazebo>
     <!-- LEFT WHEEL LINK -->
     <joint name="left_wheel_joint" type="continuous">
@@ -91,4 +93,7 @@
         </xacro:inertial_cylinder>
     </link>
+    <gazebo reference="left_wheel">
+        <material>Gazebo/Black</material>
+    </gazebo>
     <!-- RIGHT WHEEL LINK -->
     <joint name="right_wheel_joint" type="continuous">
@@ -114,4 +119,7 @@
         </xacro:inertial_cylinder>
     </link>
+    <gazebo reference="right_wheel">
+        <material>Gazebo/Red</material>
+    </gazebo>
     <!-- CASTER WHEEL LINK -->
     <joint name="caster_wheel_joint" type="fixed">
@@ -136,3 +144,8 @@
         </xacro:inertial_sphere>
     </link>
+    <gazebo reference="caster_wheel">
+        <material>Gazebo/Black</material>
+        <mu1 value="1" />
+        <mu2 value="1" />
+    </gazebo>
 </robot>
