Commit message: lidar is working

File: description/lidar.xacro (robot description, xacro)
@@ -5,5 +5,5 @@
         <child link="laser_frame"/>
         <!-- <origin xyz="0.122 0 0.212" rpy="0 0 0"/> -->
-        <origin xyz="0.1 0 0.175" rpy="0 0 0"/>
+        <origin xyz="0.1 0 0.158" rpy="0 0 0"/>
     </joint>
     <link name="laser_frame">
@@ -30,3 +30,33 @@
         </xacro:inertial_cylinder> -->
     </link>
+    <gazebo reference="laser_frame">
+        <material>Gazebo/Black</material>
+        <sensor name="laser" type="ray">
+            <pose> 0 0 0 0 0 0 </pose>
+            <visualize>true</visualize>
+            <update_rate>10</update_rate>
+            <ray>
+                <scan>
+                    <horizontal>
+                        <samples>360</samples>
+                        <resolution>1</resolution>
+                        <min_angle>-3.14</min_angle>
+                        <max_angle>3.14</max_angle>
+                    </horizontal>
+                </scan>
+                <range>
+                    <min>0.3</min>
+                    <max>12</max>
+                    <resolution>0.01</resolution>
+                </range>
+            </ray>
+            <plugin name="laser_controller" filename="libgazebo_ros_ray_sensor.so">
+                <ros>
+                    <argument>~/out:=scan</argument>
+                </ros>
+                <output_type>sensor_msgs/LaserScan</output_type>
+                <frame_name>laser_frame</frame_name>
+            </plugin>
+        </sensor>
+    </gazebo>
 </robot>

File: description/robot.urdf.xacro (robot description, xacro)
@@ -3,4 +3,5 @@
     <xacro:include filename="gazebo_control.xacro"/>
     <xacro:include filename="robot_core.xacro" />
+    <xacro:include filename="lidar.xacro"/>
     <!-- <xacro:include filename="gazebo.xacro"/> -->
 </robot>

File: description/robot_core.xacro (robot description, xacro)
@@ -1,4 +1,3 @@
 <?xml version="1.0"?>
-<!-- <robot xmlns:xacro="http://www.ros.org/wiki/xacro" name="robot"> -->
 <robot xmlns:xacro="http://www.ros.org/wiki/xacro">
     <xacro:include filename="inertial_macros.xacro"/>
@@ -55,5 +54,5 @@
                 <box size="${chassis_length} ${chassis_width} ${chassis_height}"/>
             </geometry>
-            <material name="red"/>
+            <material name="orange"/>
         </visual>
         <collision>
@@ -146,6 +145,6 @@
     <gazebo reference="caster_wheel">
         <material>Gazebo/Black</material>
-        <mu1 value="1" />
-        <mu2 value="1" />
+        <mu1 value="0.01" />
+        <mu2 value="0.01" />
     </gazebo>
 </robot>
